Commit message: model spawn success

File: factomove_description/urdf/factomove.xacro (robot description, xacro)
@@ -31,5 +31,5 @@
       <geometry>
         <mesh
-          filename="package://factomove/meshes/base_link.STL" />
+          filename="package://factomove_description/meshes/base_link.STL" />
       </geometry>
       <material
@@ -45,5 +45,5 @@
       <geometry>
         <mesh
-          filename="package://factomove/meshes/base_link.STL" />
+          filename="package://factomove_description/meshes/base_link.STL" />
       </geometry>
     </collision>
@@ -71,19 +71,19 @@
       <geometry>
         <mesh
-          filename="package://factomove/meshes/mid_left_wheel_link.STL" />
-      </geometry>
-      <material
-        name="">
-        <color
-          rgba="0.79216 0.81961 0.93333 1" />
-      </material>
-    </visual>
-    <collision>
-      <origin
-        xyz="0 0 0"
-        rpy="0 0 0" />
-      <geometry>
-        <mesh
-          filename="package://factomove/meshes/mid_left_wheel_link.STL" />
+          filename="package://factomove_description/meshes/mid_left_wheel_link.STL" />
+      </geometry>
+      <material
+        name="">
+        <color
+          rgba="0.79216 0.81961 0.93333 1" />
+      </material>
+    </visual>
+    <collision>
+      <origin
+        xyz="0 0 0"
+        rpy="0 0 0" />
+      <geometry>
+        <mesh
+          filename="package://factomove_description/meshes/mid_left_wheel_link.STL" />
       </geometry>
     </collision>
@@ -130,19 +130,19 @@
       <geometry>
         <mesh
-          filename="package://factomove/meshes/mid_right_wheel_link.STL" />
-      </geometry>
-      <material
-        name="">
-        <color
-          rgba="0.79216 0.81961 0.93333 1" />
-      </material>
-    </visual>
-    <collision>
-      <origin
-        xyz="0 0 0"
-        rpy="0 0 0" />
-      <geometry>
-        <mesh
-          filename="package://factomove/meshes/mid_right_wheel_link.STL" />
+          filename="package://factomove_description/meshes/mid_right_wheel_link.STL" />
+      </geometry>
+      <material
+        name="">
+        <color
+          rgba="0.79216 0.81961 0.93333 1" />
+      </material>
+    </visual>
+    <collision>
+      <origin
+        xyz="0 0 0"
+        rpy="0 0 0" />
+      <geometry>
+        <mesh
+          filename="package://factomove_description/meshes/mid_right_wheel_link.STL" />
       </geometry>
     </collision>
@@ -189,5 +189,5 @@
       <geometry>
         <mesh
-          filename="package://factomove/meshes/front_left_keeper_link.STL" />
+          filename="package://factomove_description/meshes/front_left_keeper_link.STL" />
       </geometry>
       <material
@@ -203,5 +203,5 @@
       <geometry>
         <mesh
-          filename="package://factomove/meshes/front_left_keeper_link.STL" />
+          filename="package://factomove_description/meshes/front_left_keeper_link.STL" />
       </geometry>
     </collision>
@@ -248,19 +248,19 @@
       <geometry>
         <mesh
-          filename="package://factomove/meshes/front_left_wheel_link.STL" />
-      </geometry>
-      <material
-        name="">
-        <color
-          rgba="0.79216 0.81961 0.93333 1" />
-      </material>
-    </visual>
-    <collision>
-      <origin
-        xyz="0 0 0"
-        rpy="0 0 0" />
-      <geometry>
-        <mesh
-          filename="package://factomove/meshes/front_left_wheel_link.STL" />
+          filename="package://factomove_description/meshes/front_left_wheel_link.STL" />
+      </geometry>
+      <material
+        name="">
+        <color
+          rgba="0.79216 0.81961 0.93333 1" />
+      </material>
+    </visual>
+    <collision>
+      <origin
+        xyz="0 0 0"
+        rpy="0 0 0" />
+      <geometry>
+        <mesh
+          filename="package://factomove_description/meshes/front_left_wheel_link.STL" />
       </geometry>
     </collision>
@@ -307,19 +307,19 @@
       <geometry>
         <mesh
-          filename="package://factomove/meshes/front_right_keeper_link.STL" />
-      </geometry>
-      <material
-        name="">
-        <color
-          rgba="0.79216 0.81961 0.93333 1" />
-      </material>
-    </visual>
-    <collision>
-      <origin
-        xyz="0 0 0"
-        rpy="0 0 0" />
-      <geometry>
-        <mesh
-          filename="package://factomove/meshes/front_right_keeper_link.STL" />
+          filename="package://factomove_description/meshes/front_right_keeper_link.STL" />
+      </geometry>
+      <material
+        name="">
+        <color
+          rgba="0.79216 0.81961 0.93333 1" />
+      </material>
+    </visual>
+    <collision>
+      <origin
+        xyz="0 0 0"
+        rpy="0 0 0" />
+      <geometry>
+        <mesh
+          filename="package://factomove_description/meshes/front_right_keeper_link.STL" />
       </geometry>
     </collision>
@@ -366,19 +366,19 @@
       <geometry>
         <mesh
-          filename="package://factomove/meshes/front_right_wheel_link.STL" />
-      </geometry>
-      <material
-        name="">
-        <color
-          rgba="0.79216 0.81961 0.93333 1" />
-      </material>
-    </visual>
-    <collision>
-      <origin
-        xyz="0 0 0"
-        rpy="0 0 0" />
-      <geometry>
-        <mesh
-          filename="package://factomove/meshes/front_right_wheel_link.STL" />
+          filename="package://factomove_description/meshes/front_right_wheel_link.STL" />
+      </geometry>
+      <material
+        name="">
+        <color
+          rgba="0.79216 0.81961 0.93333 1" />
+      </material>
+    </visual>
+    <collision>
+      <origin
+        xyz="0 0 0"
+        rpy="0 0 0" />
+      <geometry>
+        <mesh
+          filename="package://factomove_description/meshes/front_right_wheel_link.STL" />
       </geometry>
     </collision>
@@ -425,19 +425,19 @@
       <geometry>
         <mesh
-          filename="package://factomove/meshes/back_left_keeper_link.STL" />
-      </geometry>
-      <material
-        name="">
-        <color
-          rgba="0.79216 0.81961 0.93333 1" />
-      </material>
-    </visual>
-    <collision>
-      <origin
-        xyz="0 0 0"
-        rpy="0 0 0" />
-      <geometry>
-        <mesh
-          filename="package://factomove/meshes/back_left_keeper_link.STL" />
+          filename="package://factomove_description/meshes/back_left_keeper_link.STL" />
+      </geometry>
+      <material
+        name="">
+        <color
+          rgba="0.79216 0.81961 0.93333 1" />
+      </material>
+    </visual>
+    <collision>
+      <origin
+        xyz="0 0 0"
+        rpy="0 0 0" />
+      <geometry>
+        <mesh
+          filename="package://factomove_description/meshes/back_left_keeper_link.STL" />
       </geometry>
     </collision>
@@ -484,19 +484,19 @@
       <geometry>
         <mesh
-          filename="package://factomove/meshes/back_left_wheel_link.STL" />
-      </geometry>
-      <material
-        name="">
-        <color
-          rgba="0.79216 0.81961 0.93333 1" />
-      </material>
-    </visual>
-    <collision>
-      <origin
-        xyz="0 0 0"
-        rpy="0 0 0" />
-      <geometry>
-        <mesh
-          filename="package://factomove/meshes/back_left_wheel_link.STL" />
+          filename="package://factomove_description/meshes/back_left_wheel_link.STL" />
+      </geometry>
+      <material
+        name="">
+        <color
+          rgba="0.79216 0.81961 0.93333 1" />
+      </material>
+    </visual>
+    <collision>
+      <origin
+        xyz="0 0 0"
+        rpy="0 0 0" />
+      <geometry>
+        <mesh
+          filename="package://factomove_description/meshes/back_left_wheel_link.STL" />
       </geometry>
     </collision>
@@ -543,19 +543,19 @@
       <geometry>
         <mesh
-          filename="package://factomove/meshes/back_right_keeper_link.STL" />
-      </geometry>
-      <material
-        name="">
-        <color
-          rgba="0.79216 0.81961 0.93333 1" />
-      </material>
-    </visual>
-    <collision>
-      <origin
-        xyz="0 0 0"
-        rpy="0 0 0" />
-      <geometry>
-        <mesh
-          filename="package://factomove/meshes/back_right_keeper_link.STL" />
+          filename="package://factomove_description/meshes/back_right_keeper_link.STL" />
+      </geometry>
+      <material
+        name="">
+        <color
+          rgba="0.79216 0.81961 0.93333 1" />
+      </material>
+    </visual>
+    <collision>
+      <origin
+        xyz="0 0 0"
+        rpy="0 0 0" />
+      <geometry>
+        <mesh
+          filename="package://factomove_description/meshes/back_right_keeper_link.STL" />
       </geometry>
     </collision>
@@ -602,19 +602,19 @@
       <geometry>
         <mesh
-          filename="package://factomove/meshes/back_right_wheel_link.STL" />
-      </geometry>
-      <material
-        name="">
-        <color
-          rgba="0.79216 0.81961 0.93333 1" />
-      </material>
-    </visual>
-    <collision>
-      <origin
-        xyz="0 0 0"
-        rpy="0 0 0" />
-      <geometry>
-        <mesh
-          filename="package://factomove/meshes/back_right_wheel_link.STL" />
+          filename="package://factomove_description/meshes/back_right_wheel_link.STL" />
+      </geometry>
+      <material
+        name="">
+        <color
+          rgba="0.79216 0.81961 0.93333 1" />
+      </material>
+    </visual>
+    <collision>
+      <origin
+        xyz="0 0 0"
+        rpy="0 0 0" />
+      <geometry>
+        <mesh
+          filename="package://factomove_description/meshes/back_right_wheel_link.STL" />
       </geometry>
     </collision>
@@ -641,5 +641,5 @@
   <joint name="scan_joint" type="fixed">
     <axis xyz="0 1 0" />
-    <origin xyz="0 0 0.001" rpy="0 0 0"/>
+    <origin xyz="0 0 0.025" rpy="0 0 0"/>
     <parent link="base_link"/>
     <child link="base_scan"/>
@@ -649,12 +649,12 @@
     	<origin xyz="0 0 0" rpy="0 0 0"/>
       	<geometry>
-    		<box size="0.1 0.1 0.1"/>
+    		<cylinder length="0.05" radius="0.02"/>
       	</geometry>
     </collision>
     <visual>
-      	<origin xyz="0 0 0" rpy="0 0 0"/>
+      	<origin xyz="0 0 -0.015" rpy="0 0 0"/>
       	<geometry>
-        	 <!-- <mesh filename="package://factomove_description/meshes/hokuyo.dae"/>  -->
-			<cylinder length="0.1" radius="0.15"/>
+        	 <mesh filename="package://factomove_description/meshes/hokuyo.dae"/>
+			<!-- <cylinder length="0.05" radius="0.05"/> -->
       	</geometry>
     </visual>

Commit message: Add inetl realsense_d435

File: factomove_description/urdf/factomove.xacro (robot description, xacro)
@@ -1,5 +1,9 @@
 <?xml version="1.0" encoding="utf-8"?>
 <robot name="factomove" xmlns:xacro="http://www.ros.org/wiki/xacro">
-<xacro:include filename="$(find factomove_description)/urdf/factomove.gazebo"/>
+<xacro:include filename="$(find factomove_description)/urdf/factomove.gazebo.xacro"/>
+<xacro:include filename="$(find realsense2_description)/urdf/_d435.urdf.xacro" />
+<xacro:sensor_d435 name="realsense_d435" parent="base_link" >
+  <origin xyz="0.40 0 0" rpy="0 0 0" />
+</xacro:sensor_d435>
 <link name="base_footprint">
 </link>

Commit message: changed realsense pos

File: factomove_description/urdf/factomove.xacro (robot description, xacro)
@@ -4,5 +4,5 @@
 <xacro:include filename="$(find realsense2_description)/urdf/_d435.urdf.xacro" />
 <xacro:sensor_d435 name="realsense_d435" parent="base_link" >
-  <origin xyz="0.40 0 0" rpy="0 0 0" />
+  <origin xyz="0.36 0 -0.025" rpy="0 0 0" />
 </xacro:sensor_d435>
 <link name="base_footprint">
