Commit message: Add xacro files

File: factomove_description/urdf/factomove.gazebo.xacro (robot description, xacro)
@@ -1,88 +1,11 @@
 <?xml version="1.0"?>
-<robot xmlns:xacro="http://ros.org/wiki/xacro">
-<!-- <gazebo>
-<gazebo reference="mid_left_wheel_link">
-    <mu1>0.1</mu1>
-    <mu2>0.1</mu2>
-    <kp>500000.0</kp>
-    <kd>10.0</kd>
-    <minDepth>0.001</minDepth>
-    <maxVel>0.1</maxVel>
-    <fdir1>1 0 0</fdir1>
-    <material>Gazebo/FlatBlack</material>
-</gazebo>
-<gazebo reference="mid_right_wheel_link">
-    <mu1>0.1</mu1>
-    <mu2>0.1</mu2>
-    <kp>500000.0</kp>
-    <kd>10.0</kd>
-    <minDepth>0.001</minDepth>
-    <maxVel>0.1</maxVel>
-    <fdir1>1 0 0</fdir1>
-    <material>Gazebo/FlatBlack</material>
-</gazebo> -->
-<!-- <gazebo reference="front_left_wheel_link">
-</gazebo>
-<gazebo reference="back_left_wheel_link">
-</gazebo>
-<gazebo reference="front_right_wheel_link">
-</gazebo>
-<gazebo reference="back_right_wheel_link">
-</gazebo> -->
-<xacro:include filename="$(find realsense2_description)/urdf/_d435.gazebo.xacro" />
-  <gazebo>
-    <plugin name="factomove_controller" filename="libgazebo_ros_diff_drive.so">
-      <commandTopic>cmd_vel</commandTopic>
-      <odometryTopic>odom</odometryTopic>
-      <odometryFrame>odom</odometryFrame>
-      <odometrySource>world</odometrySource>
-      <publishOdomTF>true</publishOdomTF>
-      <robotBaseFrame>base_footprint</robotBaseFrame>
-      <publishWheelTF>false</publishWheelTF>
-      <publishTf>true</publishTf>
-      <publishWheelJointState>true</publishWheelJointState>
-      <legacyMode>false</legacyMode>
-      <updateRate>30</updateRate>
-      <leftJoint>mid_left_wheel_joint</leftJoint>
-      <rightJoint>mid_right_wheel_joint</rightJoint>
-      <wheelSeparation>0.5583</wheelSeparation>
-      <wheelDiameter>0.16</wheelDiameter>
-      <wheelAcceleration>1</wheelAcceleration>
-      <wheelTorque>100</wheelTorque>
-      <rosDebugLevel>na</rosDebugLevel>
-    </plugin>
-  </gazebo>
-<!-- hokuyo -->
-  <gazebo reference="base_scan">
-   <material>Gazebo/FlatBlack</material>
-    <sensor type="ray" name="lds_lfcd_sensor">
-      <pose>0 0 0 0 0 0</pose>
-      <visualize>true</visualize>
-      <update_rate>5</update_rate>
-      <ray>
-        <scan>
-          <horizontal>
-            <samples>360</samples>
-            <resolution>1</resolution>
-            <min_angle>0.0</min_angle>
-            <max_angle>6.28319</max_angle>
-          </horizontal>
-        </scan>
-        <range>
-          <min>0.03</min>
-          <max>7</max>
-          <resolution>0.015</resolution>
-        </range>
-        <noise>
-          <type>gaussian</type>
-          <mean>0.0</mean>
-          <stddev>0.01</stddev>
-        </noise>
-      </ray>
-      <plugin name="gazebo_ros_lds_lfcd_controller" filename="libgazebo_ros_laser.so">
-        <topicName>scan</topicName>
-        <frameName>base_scan</frameName>
-      </plugin>
-    </sensor>
-  </gazebo>
+<robot xmlns:xacro="http://www.ros.org/wiki/xacro">
+  <xacro:include filename="$(find realsense2_description)/urdf/_d435.urdf.xacro"/>
+  <xacro:include filename="$(find realsense2_description)/urdf/_d435.gazebo.xacro"/>
+  <xacro:sensor_d435 name="realsense_d435" parent="base_link" >
+    <origin xyz="0.36 0 -0.025" rpy="0 0 0" />
+  </xacro:sensor_d435>
+  <xacro:include filename="$(find factomove_description)/urdf/hokuyo_lidar.urdf.xacro"/>
+  <xacro:include filename="$(find factomove_description)/urdf/hokuyo_lidar.gazebo.xacro"/>
+  <xacro:include filename="$(find factomove_description)/urdf/diff_drive_controller.gazebo.xacro"/>
 </robot>

File: factomove_description/urdf/factomove.xacro (robot description, xacro)
@@ -1,671 +1,5 @@
-<?xml version="1.0" encoding="utf-8"?>
-<robot name="factomove" xmlns:xacro="http://www.ros.org/wiki/xacro">
+<?xml version="1.0"?>
+<robot xmlns:xacro="http://www.ros.org/wiki/xacro" name="factomove">
+<xacro:include filename="$(find factomove_description)/urdf/factomove.urdf.xacro"/>
 <xacro:include filename="$(find factomove_description)/urdf/factomove.gazebo.xacro"/>
-<xacro:include filename="$(find realsense2_description)/urdf/_d435.urdf.xacro" />
-<xacro:sensor_d435 name="realsense_d435" parent="base_link" >
-  <origin xyz="0.36 0 -0.025" rpy="0 0 0" />
-</xacro:sensor_d435>
-<link name="base_footprint">
-</link>
-<joint name="base_joint" type="fixed">
-	<parent link="base_footprint"/>
-	<child link="base_link"/>
-      <origin xyz="0.0 0.0 0.0" rpy="0 0 0"/>
-</joint>
-  <link
-    name="base_link">
-    <inertial>
-      <origin
-        xyz="6.1085E-11 7.0637E-11 -0.058359"
-        rpy="0 0 0" />
-      <mass
-        value="11.93" />
-      <inertia
-        ixx="0.24655"
-        ixy="1.0146E-10"
-        ixz="-7.2198E-14"
-        iyy="0.44294"
-        iyz="1.8415E-13"
-        izz="0.61972" />
-    </inertial>
-    <visual>
-      <origin
-        xyz="0 0 0"
-        rpy="0 0 0" />
-      <geometry>
-        <mesh
-          filename="package://factomove_description/meshes/base_link.STL" />
-      </geometry>
-      <material
-        name="">
-        <color
-          rgba="1 1 1 1" />
-      </material>
-    </visual>
-    <collision>
-      <origin
-        xyz="0 0 0"
-        rpy="0 0 0" />
-      <geometry>
-        <mesh
-          filename="package://factomove_description/meshes/base_link.STL" />
-      </geometry>
-    </collision>
-  </link>
-  <link
-    name="mid_left_wheel_link">
-    <inertial>
-      <origin
-        xyz="-6.3781E-06 -0.027802 1.0717E-06"
-        rpy="0 0 0" />
-      <mass
-        value="1.0785" />
-      <inertia
-        ixx="0.0019839"
-        ixy="-3.8726E-07"
-        ixz="-5.7089E-09"
-        iyy="0.0033904"
-        iyz="6.5067E-08"
-        izz="0.0019839" />
-    </inertial>
-    <visual>
-      <origin
-        xyz="0 0 0"
-        rpy="0 0 0" />
-      <geometry>
-        <mesh
-          filename="package://factomove_description/meshes/mid_left_wheel_link.STL" />
-      </geometry>
-      <material
-        name="">
-        <color
-          rgba="0.79216 0.81961 0.93333 1" />
-      </material>
-    </visual>
-    <collision>
-      <origin
-        xyz="0 0 0"
-        rpy="0 0 0" />
-      <geometry>
-        <mesh
-          filename="package://factomove_description/meshes/mid_left_wheel_link.STL" />
-      </geometry>
-    </collision>
-  </link>
-  <joint
-    name="mid_left_wheel_joint"
-    type="continuous">
-    <origin
-      xyz="0 0.224 -0.141"
-      rpy="0 0 0" />
-    <parent
-      link="base_link" />
-    <child
-      link="mid_left_wheel_link" />
-    <axis
-      xyz="0 1 0" />
-    <limit
-      effort="10"
-      velocity="10" />
-    <dynamics
-      damping="0.1"
-      friction="0.1" />
-  </joint>
-  <link
-    name="mid_right_wheel_link">
-    <inertial>
-      <origin
-        xyz="3.043E-06 0.027802 -5.7069E-06"
-        rpy="0 0 0" />
-      <mass
-        value="1.0785" />
-      <inertia
-        ixx="0.0019839"
-        ixy="-1.8476E-07"
-        ixz="-1.4505E-08"
-        iyy="0.0033904"
-        iyz="3.465E-07"
-        izz="0.0019839" />
-    </inertial>
-    <visual>
-      <origin
-        xyz="0 0 0"
-        rpy="0 0 0" />
-      <geometry>
-        <mesh
-          filename="package://factomove_description/meshes/mid_right_wheel_link.STL" />
-      </geometry>
-      <material
-        name="">
-        <color
-          rgba="0.79216 0.81961 0.93333 1" />
-      </material>
-    </visual>
-    <collision>
-      <origin
-        xyz="0 0 0"
-        rpy="0 0 0" />
-      <geometry>
-        <mesh
-          filename="package://factomove_description/meshes/mid_right_wheel_link.STL" />
-      </geometry>
-    </collision>
-  </link>
-  <joint
-    name="mid_right_wheel_joint"
-    type="continuous">
-    <origin
-      xyz="0 -0.224 -0.141"
-      rpy="0 0 0" />
-    <parent
-      link="base_link" />
-    <child
-      link="mid_right_wheel_link" />
-    <axis
-      xyz="0 1 0" />
-    <limit
-      effort="10"
-      velocity="10" />
-    <dynamics
-      damping="0.1"
-      friction="0.1" />
-  </joint>
-  <link
-    name="front_left_keeper_link">
-    <inertial>
-      <origin
-        xyz="-0.0266276705620659 0.000666352830324346 -0.0393449495275665"
-        rpy="0 0 0" />
-      <mass
-        value="0.102809337693291" />
-      <inertia
-        ixx="0.000195021798600733"
-        ixy="-1.2184873072082E-07"
-        ixz="-4.0809835332173E-05"
-        iyy="0.000167393233669256"
-        iyz="9.24624427261228E-08"
-        izz="0.000195015527031851" />
-    </inertial>
-    <visual>
-      <origin
-        xyz="0 0 0"
-        rpy="0 0 0" />
-      <geometry>
-        <mesh
-          filename="package://factomove_description/meshes/front_left_keeper_link.STL" />
-      </geometry>
-      <material
-        name="">
-        <color
-          rgba="0.792156862745098 0.819607843137255 0.933333333333333 1" />
-      </material>
-    </visual>
-    <collision>
-      <origin
-        xyz="0 0 0"
-        rpy="0 0 0" />
-      <geometry>
-        <mesh
-          filename="package://factomove_description/meshes/front_left_keeper_link.STL" />
-      </geometry>
-    </collision>
-  </link>
-  <joint
-    name="front_left_keeper_joint"
-    type="continuous">
-    <origin
-      xyz="0.2925 0.17 -0.040635"
-      rpy="0 0 0" />
-    <parent
-      link="base_link" />
-    <child
-      link="front_left_keeper_link" />
-    <axis
-      xyz="0 0 -1" />
-    <limit
-      effort="10"
-      velocity="10" />
-    <dynamics
-      damping="0.1"
-      friction="0.1" />
-  </joint>
-  <link
-    name="front_left_wheel_link">
-    <inertial>
-      <origin
-        xyz="-3.8734E-09 1.1658E-09 3.0966E-09"
-        rpy="0 0 0" />
-      <mass
-        value="0.67052" />
-      <inertia
-        ixx="0.0015386"
-        ixy="4.1231E-06"
-        ixz="-5.9599E-12"
-        iyy="0.0028064"
-        iyz="2.5984E-12"
-        izz="0.0015386" />
-    </inertial>
-    <visual>
-      <origin
-        xyz="0 0 0"
-        rpy="0 0 0" />
-      <geometry>
-        <mesh
-          filename="package://factomove_description/meshes/front_left_wheel_link.STL" />
-      </geometry>
-      <material
-        name="">
-        <color
-          rgba="0.79216 0.81961 0.93333 1" />
-      </material>
-    </visual>
-    <collision>
-      <origin
-        xyz="0 0 0"
-        rpy="0 0 0" />
-      <geometry>
-        <mesh
-          filename="package://factomove_description/meshes/front_left_wheel_link.STL" />
-      </geometry>
-    </collision>
-  </link>
-  <joint
-    name="front_left_wheel_joint"
-    type="continuous">
-    <origin
-      xyz="-0.053 0.00017237 -0.10037"
-      rpy="0 0 0" />
-    <parent
-      link="front_left_keeper_link" />
-    <child
-      link="front_left_wheel_link" />
-    <axis
-      xyz="-0.0032522 -0.99999 0" />
-    <limit
-      effort="10"
-      velocity="10" />
-    <dynamics
-      damping="0.1"
-      friction="0.1" />
-  </joint>
-  <link
-    name="front_right_keeper_link">
-    <inertial>
-      <origin
-        xyz="-0.026628 0.00066635 -0.039345"
-        rpy="0 0 0" />
-      <mass
-        value="0.10281" />
-      <inertia
-        ixx="0.00019502"
-        ixy="-1.2185E-07"
-        ixz="-4.081E-05"
-        iyy="0.00016739"
-        iyz="9.2462E-08"
-        izz="0.00019502" />
-    </inertial>
-    <visual>
-      <origin
-        xyz="0 0 0"
-        rpy="0 0 0" />
-      <geometry>
-        <mesh
-          filename="package://factomove_description/meshes/front_right_keeper_link.STL" />
-      </geometry>
-      <material
-        name="">
-        <color
-          rgba="0.79216 0.81961 0.93333 1" />
-      </material>
-    </visual>
-    <collision>
-      <origin
-        xyz="0 0 0"
-        rpy="0 0 0" />
-      <geometry>
-        <mesh
-          filename="package://factomove_description/meshes/front_right_keeper_link.STL" />
-      </geometry>
-    </collision>
-  </link>
-  <joint
-    name="front_right_keeper_joint"
-    type="continuous">
-    <origin
-      xyz="0.2925 -0.17 -0.040635"
-      rpy="0 0 0" />
-    <parent
-      link="base_link" />
-    <child
-      link="front_right_keeper_link" />
-    <axis
-      xyz="0 0 -1" />
-    <limit
-      effort="10"
-      velocity="10" />
-    <dynamics
-      damping="0.1"
-      friction="0.1" />
-  </joint>
-  <link
-    name="front_right_wheel_link">
-    <inertial>
-      <origin
-        xyz="-3.8734E-09 1.1658E-09 3.0966E-09"
-        rpy="0 0 0" />
-      <mass
-        value="0.67052" />
-      <inertia
-        ixx="0.0015386"
-        ixy="4.1231E-06"
-        ixz="-5.9599E-12"
-        iyy="0.0028064"
-        iyz="2.5984E-12"
-        izz="0.0015386" />
-    </inertial>
-    <visual>
-      <origin
-        xyz="0 0 0"
-        rpy="0 0 0" />
-      <geometry>
-        <mesh
-          filename="package://factomove_description/meshes/front_right_wheel_link.STL" />
-      </geometry>
-      <material
-        name="">
-        <color
-          rgba="0.79216 0.81961 0.93333 1" />
-      </material>
-    </visual>
-    <collision>
-      <origin
-        xyz="0 0 0"
-        rpy="0 0 0" />
-      <geometry>
-        <mesh
-          filename="package://factomove_description/meshes/front_right_wheel_link.STL" />
-      </geometry>
-    </collision>
-  </link>
-  <joint
-    name="front_right_wheel_joint"
-    type="continuous">
-    <origin
-      xyz="-0.053 0.00017237 -0.10037"
-      rpy="0 0 0" />
-    <parent
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