Commit message: mapping in real life

File: factomove_description/urdf/factomove.urdf.xacro (robot description, xacro)
@@ -1,10 +1,9 @@
 <?xml version="1.0"?>
-<robot xmlns:xacro="http://www.ros.org/wiki/xacro">
-  <link name="base_footprint">
-  </link>
+<robot name="factomove" xmlns:xacro="http://www.ros.org/wiki/xacro">
+  <link name="base_footprint"/>
   <joint name="base_joint" type="fixed">
-      <parent link="base_footprint"/>
-      <child link="base_link"/>
-          <origin xyz="0.0 0.0 0.0" rpy="0 0 0"/>
+    <parent link="base_footprint"/>
+    <child link="base_link" />
+    <origin xyz="0 0 0.010" rpy="0 0 0"/>
   </joint>
   <link
@@ -638,3 +637,29 @@
       friction="0.1" />
   </joint>
+  <joint name="scan_joint" type="fixed">
+    <parent link="base_link"/>
+    <child link="base_scan"/>
+    <origin xyz="-0.064 0 0.122" rpy="0 0 0"/>
+  </joint>
+  <link name="base_scan">
+    <visual>
+      <origin xyz="0 0 0" rpy="0 0 0"/>
+      <geometry>
+        <mesh filename="package://factomove_description/meshes/hokuyo.dae"/>
+      </geometry>
+    </visual>
+    <collision>
+      <origin xyz="0.015 0 -0.0065" rpy="0 0 0"/>
+      <geometry>
+        <cylinder length="0.0315" radius="0.055"/>
+      </geometry>
+    </collision>
+    <inertial>
+      <mass value="0.114" />
+      <origin xyz="0 0 0" />
+      <inertia ixx="0.001" ixy="0.0" ixz="0.0"
+               iyy="0.001" iyz="0.0"
+               izz="0.001" />
+    </inertial>
+  </link>
 </robot>

Commit message: some_work

File: factomove_description/urdf/factomove.urdf.xacro (robot description, xacro)
@@ -640,5 +640,5 @@
     <parent link="base_link"/>
     <child link="base_scan"/>
-    <origin xyz="-0.064 0 0.122" rpy="0 0 0"/>
+    <origin xyz="0.3 0 0.025" rpy="0 0 0"/>
   </joint>
   <link name="base_scan">

File: factomove_description/urdf/hokuyo_lidar.urdf.xacro (robot description, xacro)
@@ -22,5 +22,5 @@
   <joint name="scan_joint" type="fixed">
     <axis xyz="0 1 0" />
-    <origin xyz="0 0 0.025" rpy="0 0 0"/>
+    <origin xyz="0.3 0 0.025" rpy="0 0 0"/>
     <parent link="base_link"/>
     <child link="base_scan"/>

Commit message: added new urdf and minor fixed move_base

File: factomove_description/urdf/factomove.urdf.xacro (robot description, xacro)
@@ -1,3 +1,3 @@
-<?xml version="1.0"?>
+<?xml version="1.0" encoding="utf-8"?>
 <robot name="factomove" xmlns:xacro="http://www.ros.org/wiki/xacro">
   <link name="base_footprint"/>
@@ -9,18 +9,4 @@
   <link
     name="base_link">
-    <inertial>
-      <origin
-        xyz="6.1085E-11 7.0637E-11 -0.058359"
-        rpy="0 0 0" />
-      <mass
-        value="11.93" />
-      <inertia
-        ixx="0.24655"
-        ixy="1.0146E-10"
-        ixz="-7.2198E-14"
-        iyy="0.44294"
-        iyz="1.8415E-13"
-        izz="0.61972" />
-    </inertial>
     <visual>
       <origin
@@ -34,5 +20,5 @@
         name="">
         <color
-          rgba="1 1 1 1" />
+          rgba="0.79216 0.81961 0.93333 1" />
       </material>
     </visual>
@@ -48,19 +34,5 @@
   </link>
   <link
-    name="left_wheel">
-    <inertial>
-      <origin
-        xyz="-6.3781E-06 -0.027802 1.0717E-06"
-        rpy="0 0 0" />
-      <mass
-        value="1.0785" />
-      <inertia
-        ixx="0.0019839"
-        ixy="-3.8726E-07"
-        ixz="-5.7089E-09"
-        iyy="0.0033904"
-        iyz="6.5067E-08"
-        izz="0.0019839" />
-    </inertial>
+    name="right_wheel">
     <visual>
       <origin
@@ -69,10 +41,10 @@
       <geometry>
         <mesh
-          filename="package://factomove_description/meshes/mid_left_wheel_link.STL" />
+          filename="package://factomove_description/meshes/right_wheel_link.STL" />
       </geometry>
       <material
         name="">
         <color
-          rgba="0.79216 0.81961 0.93333 1" />
+          rgba="0.44706 0.47451 0.50196 1" />
       </material>
     </visual>
@@ -83,43 +55,23 @@
       <geometry>
         <mesh
-          filename="package://factomove_description/meshes/mid_left_wheel_link.STL" />
+          filename="package://factomove_description/meshes/right_wheel_link.STL" />
       </geometry>
     </collision>
   </link>
   <joint
-    name="left_wheel"
+    name="right_wheel"
     type="continuous">
     <origin
-      xyz="0 0.224 -0.141"
-      rpy="0 0 0" />
+      xyz="-0.041648 -0.19304 -0.103"
+      rpy="-1.5708 0 0" />
     <parent
       link="base_link" />
     <child
-      link="left_wheel" />
+      link="right_wheel" />
     <axis
-      xyz="0 1 0" />
-    <limit
-      effort="10"
-      velocity="10" />
-    <dynamics
-      damping="0.1"
-      friction="0.1" />
+      xyz="0 0 1" />
   </joint>
   <link
-    name="right_wheel">
-    <inertial>
-      <origin
-        xyz="3.043E-06 0.027802 -5.7069E-06"
-        rpy="0 0 0" />
-      <mass
-        value="1.0785" />
-      <inertia
-        ixx="0.0019839"
-        ixy="-1.8476E-07"
-        ixz="-1.4505E-08"
-        iyy="0.0033904"
-        iyz="3.465E-07"
-        izz="0.0019839" />
-    </inertial>
+    name="left_wheel">
     <visual>
       <origin
@@ -128,10 +80,10 @@
       <geometry>
         <mesh
-          filename="package://factomove_description/meshes/mid_right_wheel_link.STL" />
+          filename="package://factomove_description/meshes/left_wheel_link.STL" />
       </geometry>
       <material
         name="">
         <color
-          rgba="0.79216 0.81961 0.93333 1" />
+          rgba="0.44706 0.47451 0.50196 1" />
       </material>
     </visual>
@@ -142,43 +94,36 @@
       <geometry>
         <mesh
-          filename="package://factomove_description/meshes/mid_right_wheel_link.STL" />
+          filename="package://factomove_description/meshes/left_wheel_link.STL" />
       </geometry>
     </collision>
   </link>
   <joint
-    name="right_wheel"
+    name="left_wheel"
     type="continuous">
     <origin
-      xyz="0 -0.224 -0.141"
+      xyz="-0.041648 0.19296 -0.103"
+      rpy="-1.5708 0 0" />
+    <parent
+      link="base_link" />
+    <child
+      link="left_wheel" />
+    <axis
+      xyz="0 0 -1" />
+  </joint>
+    <joint
+    name="scan_joint"
+    type="fixed">
+    <origin
+      xyz="0.47473 -4.3283E-05 0.016542"
       rpy="0 0 0" />
     <parent
       link="base_link" />
     <child
-      link="right_wheel" />
+      link="base_scan" />
     <axis
-      xyz="0 1 0" />
-    <limit
-      effort="10"
-      velocity="10" />
-    <dynamics
-      damping="0.1"
-      friction="0.1" />
+      xyz="0 0 0" />
   </joint>
   <link
-    name="front_left_keeper_link">
-    <inertial>
-      <origin
-        xyz="-0.0266276705620659 0.000666352830324346 -0.0393449495275665"
-        rpy="0 0 0" />
-      <mass
-        value="0.102809337693291" />
-      <inertia
-        ixx="0.000195021798600733"
-        ixy="-1.2184873072082E-07"
-        ixz="-4.0809835332173E-05"
-        iyy="0.000167393233669256"
-        iyz="9.24624427261228E-08"
-        izz="0.000195015527031851" />
-    </inertial>
+    name="base_scan">
     <visual>
       <origin
@@ -187,10 +132,10 @@
       <geometry>
         <mesh
-          filename="package://factomove_description/meshes/front_left_keeper_link.STL" />
+          filename="package://factomove_description/meshes/base_scan.STL" />
       </geometry>
       <material
         name="">
         <color
-          rgba="0.792156862745098 0.819607843137255 0.933333333333333 1" />
+          rgba="0.44706 0.47451 0.50196 1" />
       </material>
     </visual>
@@ -201,465 +146,7 @@
       <geometry>
         <mesh
-          filename="package://factomove_description/meshes/front_left_keeper_link.STL" />
+          filename="package://factomove_description/meshes/base_scan.STL" />
       </geometry>
     </collision>
   </link>
-  <joint
-    name="front_left_keeper_joint"
-    type="continuous">
-    <origin
-      xyz="0.2925 0.17 -0.040635"
-      rpy="0 0 0" />
-    <parent
-      link="base_link" />
-    <child
-      link="front_left_keeper_link" />
-    <axis
-      xyz="0 0 -1" />
-    <limit
-      effort="10"
-      velocity="10" />
-    <dynamics
-      damping="0.1"
-      friction="0.1" />
-  </joint>
-  <link
-    name="front_left_wheel_link">
-    <inertial>
-      <origin
-        xyz="-3.8734E-09 1.1658E-09 3.0966E-09"
-        rpy="0 0 0" />
-      <mass
-        value="0.67052" />
-      <inertia
-        ixx="0.0015386"
-        ixy="4.1231E-06"
-        ixz="-5.9599E-12"
-        iyy="0.0028064"
-        iyz="2.5984E-12"
-        izz="0.0015386" />
-    </inertial>
-    <visual>
-      <origin
-        xyz="0 0 0"
-        rpy="0 0 0" />
-      <geometry>
-        <mesh
-          filename="package://factomove_description/meshes/front_left_wheel_link.STL" />
-      </geometry>
-      <material
-        name="">
-        <color
-          rgba="0.79216 0.81961 0.93333 1" />
-      </material>
-    </visual>
-    <collision>
-      <origin
-        xyz="0 0 0"
-        rpy="0 0 0" />
-      <geometry>
-        <mesh
-          filename="package://factomove_description/meshes/front_left_wheel_link.STL" />
-      </geometry>
-    </collision>
-  </link>
-  <joint
-    name="front_left_wheel_joint"
-    type="continuous">
-    <origin
-      xyz="-0.053 0.00017237 -0.10037"
-      rpy="0 0 0" />
-    <parent
-      link="front_left_keeper_link" />
-    <child
-      link="front_left_wheel_link" />
-    <axis
-      xyz="-0.0032522 -0.99999 0" />
-    <limit
-      effort="10"
-      velocity="10" />
-    <dynamics
-      damping="0.1"
-      friction="0.1" />
-  </joint>
-  <link
-    name="front_right_keeper_link">
-    <inertial>
-      <origin
-        xyz="-0.026628 0.00066635 -0.039345"
-        rpy="0 0 0" />
-      <mass
-        value="0.10281" />
-      <inertia
-        ixx="0.00019502"
-        ixy="-1.2185E-07"
-        ixz="-4.081E-05"
-        iyy="0.00016739"
-        iyz="9.2462E-08"
-        izz="0.00019502" />
-    </inertial>
-    <visual>
-      <origin
-        xyz="0 0 0"
-        rpy="0 0 0" />
-      <geometry>
-        <mesh
-          filename="package://factomove_description/meshes/front_right_keeper_link.STL" />
-      </geometry>
-      <material
-        name="">
-        <color
-          rgba="0.79216 0.81961 0.93333 1" />
-      </material>
-    </visual>
-    <collision>
-      <origin
-        xyz="0 0 0"
-        rpy="0 0 0" />
-      <geometry>
-        <mesh
-          filename="package://factomove_description/meshes/front_right_keeper_link.STL" />
-      </geometry>
-    </collision>
-  </link>
-  <joint
-    name="front_right_keeper_joint"
-    type="continuous">
-    <origin
-      xyz="0.2925 -0.17 -0.040635"
-      rpy="0 0 0" />
-    <parent
-      link="base_link" />
-    <child
-      link="front_right_keeper_link" />
-    <axis
-      xyz="0 0 -1" />
-    <limit
-      effort="10"
-      velocity="10" />
-    <dynamics
-      damping="0.1"
-      friction="0.1" />
-  </joint>
-  <link
-    name="front_right_wheel_link">
-    <inertial>
-      <origin
-        xyz="-3.8734E-09 1.1658E-09 3.0966E-09"
-        rpy="0 0 0" />
-      <mass
-        value="0.67052" />
-      <inertia
-        ixx="0.0015386"
-        ixy="4.1231E-06"
-        ixz="-5.9599E-12"
-        iyy="0.0028064"
-        iyz="2.5984E-12"
-        izz="0.0015386" />
-    </inertial>
-    <visual>
-      <origin
-        xyz="0 0 0"
-        rpy="0 0 0" />
-      <geometry>
-        <mesh
-          filename="package://factomove_description/meshes/front_right_wheel_link.STL" />
-      </geometry>
-      <material
-        name="">
-        <color
-          rgba="0.79216 0.81961 0.93333 1" />
-      </material>
-    </visual>
-    <collision>
-      <origin
-        xyz="0 0 0"
-        rpy="0 0 0" />
-      <geometry>
-        <mesh
-          filename="package://factomove_description/meshes/front_right_wheel_link.STL" />
-      </geometry>
-    </collision>
-  </link>
-  <joint
-    name="front_right_wheel_joint"
-    type="continuous">
-    <origin
-      xyz="-0.053 0.00017237 -0.10037"
-      rpy="0 0 0" />
-    <parent
-      link="front_right_keeper_link" />
-    <child
-      link="front_right_wheel_link" />
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